File: telemetry-kicad/telemetry.kicad_pcb (KiCad board)
At the start: 4 copper layers, 98 parts, among them J1 2601-1102, J2 RFPC-SMA27-F, J3 TC2030, J4 2601-1102, J5 2601-1102, J6 USB_C_Receptacle_USB2.0_16P, J7 SD_Card_Receptacle, Q1 DMP3099LQ-7, SW1 SW_NRST, SW2 SW_BOOT0, U1 LMR33610ADDAR, U10 TLC59108IPWR, U11 MCP1703T-5002E/CB, U2 ASM330LHHXG1TR, U3 MAX-M10S-00B, U4 TCAN337, U5 STM32H523RCT7, U6 TCAN337, U7 USBLC6-2SC6, U9 TLC59108IPWR, Y1 ABM8AIG-24.000MHz-8-2Z-T

Commit message: Layout progress
Parts:
- TP5: value CANH1 -> CAN1+
- TP6: value CANL1 -> CAN1-
- TP7: value CANH2 -> CAN2+
- TP8: value CANL2 -> CAN2-
- moved LED5 159.3 mm to (90.0, 72.8), turned to 90 degrees
- moved LED4 156.6 mm to (93.5, 73.0), turned to 90 degrees
- moved C33 154.5 mm to (94.8, 84.2), turned to 0 degrees
- moved LED3 153.6 mm to (97.2, 72.8), turned to 90 degrees
- moved LED2 150.9 mm to (101.0, 73.0), turned to 90 degrees
- moved LED1 148.2 mm to (104.8, 73.0), turned to 90 degrees
- moved C34 147.3 mm to (94.8, 67.8), turned to 0 degrees
- moved U9 140.3 mm to (100.8, 80.5), turned to 180 degrees
- moved C32 140.2 mm to (97.5, 47.2), turned to 0 degrees
- moved D6 140.0 mm to (97.5, 53.1), turned to -90 degrees
- moved U10 134.0 mm to (101.0, 64.8), turned to 180 degrees
- moved U11 130.9 mm to (102.2, 48.4), turned to 180 degrees
- moved R21 129.0 mm to (89.8, 84.0)
- moved R12 129.0 mm to (89.8, 77.0)
- moved R13 129.0 mm to (89.8, 80.5)
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Connections:
- net /CANH1 renamed /CAN1+
- net /CANH2 renamed /CAN2+
- net /CANL1 renamed /CAN1-
- net /CANL2 renamed /CAN2-
Routing:
- net SDA_LED: track 0.00 -> 29.5 mm, vias 0 -> 2
- net SCL_LED: track 0.00 -> 28.8 mm, vias 0 -> 2
- net RST_LED: track 0.00 -> 26.9 mm, vias 0 -> 2
- net NRST: track 0.00 -> 26.9 mm
- net LED8: track 0.00 -> 22.5 mm, vias 0 -> 2
- net LED6: track 0.00 -> 17.1 mm
- net LED3: track 0.00 -> 15.0 mm, vias 0 -> 2
- net LED7: track 0.00 -> 13.9 mm, vias 0 -> 2
- net LED9: track 0.00 -> 13.7 mm, vias 0 -> 2
- net LED5: track 0.00 -> 12.2 mm, vias 0 -> 2
- net LED1: track 0.00 -> 12.0 mm
- net SWDIO: track 0.00 -> 8.84 mm, vias 0 -> 2
- net SWO: track 0.00 -> 8.21 mm
- net LED0: track 0.00 -> 7.15 mm
- net SWCLK: track 0.00 -> 6.01 mm
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- added copper zone on F.Cu, net V_IN

Commit message: PCB draft complete
Parts:
- removed C28: 1uF, Capacitor_SMD:C_0805_2012Metric_Pad1.18x1.45mm_HandSolder
- moved J7 181.5 mm to (105.3, 34.2)
- moved C17 181.5 mm to (61.2, 34.8)
- moved R14 181.5 mm to (61.2, 30.0)
- moved R15 181.5 mm to (61.2, 37.2)
- moved R16 181.5 mm to (61.2, 27.5)
- moved R17 181.5 mm to (61.2, 24.8)
- moved R18 181.5 mm to (61.2, 44.2)
- moved R19 181.5 mm to (61.2, 41.8)
- moved C27 143.0 mm to (23.2, 62.5), turned to 180 degrees
- moved C26 142.5 mm to (23.2, 64.8), turned to 0 degrees
- moved U2 141.2 mm to (22.9, 59.8)
- moved J1 70.2 mm to (65.2, 82.8), turned to 0 degrees
- moved TP4 51.7 mm to (76.2, 57.2)
- moved J2 48.5 mm to (25.8, 24.0)
- moved C29 48.5 mm to (28.9, 50.2)
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Routing:
- net DI_IMU: track 0.00 -> 21.9 mm
- net INT2: track 0.00 -> 21.4 mm, vias 0 -> 2
- net SCK_IMU: track 0.00 -> 21.4 mm
- net DO_IMU: track 0.00 -> 20.2 mm, vias 0 -> 2
- net INT1: track 0.00 -> 17.2 mm
- net CS_IMU: track 0.00 -> 16.6 mm, vias 0 -> 2
- net +3.3V: track 66.1 -> 66.0 mm, vias 0 -> 3
- net GND: vias 33 -> 30
Other:
- board outline added: 94 x 83.5 mm
