File: telemetry-kicad/telemetry.kicad_pcb (KiCad board)
At the start: 4 copper layers, 72.2 x 83.5 mm, 122 parts, among them J1 2601-1102, J2 RFPC-SMA27-F, J3 TC2030, J4 2601-1102, J5 MOLEX_104031-0811, J6 2601-1102, J7 USB_C_Receptacle_USB2.0_16P, Q1 DMP3099LQ-7, Q2 MMBT3904, SW1 CJS-1200TB1, SW2 CJS-1200TB1, SW3 SW_NRST, SW4 SW_BOOT0, U1 LMR33610ADDAR, U10 LC29HBAMD, U11 USBLC6-2SC6, U12 TXS0108EPW, U2 TPS2121RUXR, U3 ASM330LHHXG1TR, U4 TCAN337, U5 LM2940CT-5.0/LF01, U6 STM32H523RCT7, U7 TCAN337, U8 TLC59108IPWR, U9 TLC59108IPWR, Y1 ABM8AIG-24.000MHz-8-2Z-T

Commit message: Finished all design, no DRC issues. Added BOM, cleaned folder
Parts:
- added H1: MountingHole_Pad, telemetry:MountingHole_3.2mm_M3_Pad, F.Cu at (17.5, 17.5)
- added H2: MountingHole_Pad, telemetry:MountingHole_3.2mm_M3_Pad, F.Cu at (88.5, 17.5)
- added H3: MountingHole_Pad, telemetry:MountingHole_3.2mm_M3_Pad, F.Cu at (17.5, 87.0)
- added H4: MountingHole_Pad, telemetry:MountingHole_3.2mm_M3_Pad, F.Cu at (88.5, 87.0)
- U3: value ASM330LHHXG1TR -> LGA14_2P5X3_STM
- moved R11 125.3 mm to (75.7, 73.5), turned to 180 degrees
- moved C2 123.7 mm to (77.9, 67.0), turned to 90 degrees
- moved R9 122.6 mm to (76.2, 75.5), turned to 90 degrees
- moved R3 119.0 mm to (79.2, 67.0), turned to 90 degrees
- moved R10 118.3 mm to (79.9, 75.5), turned to 90 degrees
- moved R12 116.2 mm to (81.2, 75.5), turned to -90 degrees
- moved TP4 114.0 mm to (63.4, 51.5)
- moved R5 112.9 mm to (78.7, 75.5), turned to -90 degrees
- moved TP2 112.8 mm to (60.1, 52.3)
- moved R2 112.4 mm to (82.4, 75.5), turned to 90 degrees
- moved R1 111.6 mm to (77.4, 75.5), turned to 90 degrees
- moved R6 109.8 mm to (82.9, 73.5)
- moved U2 107.1 mm to (78.9, 71.0)
- moved F1 103.1 mm to (77.9, 83.7), turned to 0 degrees
- moved D3 102.9 mm to (78.4, 89.3)
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Connections:
- J4 pad 1: /CAN1+ -> /CAN1-
- J4 pad 2: /CAN1+ -> /CAN1-
- J4 pad 3: /CAN1- -> /CAN1+
- J4 pad 4: /CAN1- -> /CAN1+
- J6 pad 1: /CAN2+ -> /CAN2-
- J6 pad 2: /CAN2+ -> /CAN2-
- J6 pad 3: /CAN2- -> /CAN2+
- J6 pad 4: /CAN2- -> /CAN2+
Routing:
- net SCL_LED: track 26.2 -> 86.5 mm, vias 2 -> 4
- net /VBUS: track 25.7 -> 84.2 mm
- net FLT_CAN2: track 0.00 -> 50.6 mm, vias 0 -> 4
- net FLT_CAN1: track 0.00 -> 48.2 mm, vias 0 -> 2
- net +3.3V: track 49.8 -> 96.5 mm, vias 22 -> 48
- net SIL_CAN2: track 0.00 -> 46.3 mm, vias 0 -> 4
- net RST_LED: track 24.5 -> 69.1 mm
- net RXD_CAN2: track 0.00 -> 44.5 mm, vias 0 -> 4
- net V_IN: track 15.2 -> 59.5 mm, vias 0 -> 2
- net +5V: track 0.00 -> 44.1 mm
- net TXD_CAN2: track 0.00 -> 42.7 mm, vias 0 -> 4
- net SDA_LED: track 27.0 -> 69.0 mm, vias 2 -> 6
- net D1_SD: track 0.00 -> 41.0 mm, vias 0 -> 4
- net D0_SD: track 0.00 -> 40.2 mm, vias 0 -> 4
- net RXD_CAN1: track 0.00 -> 40.1 mm
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- added copper zone on F.Cu, net +12V
- added copper zone on In2.Cu, net +3.3V
- added copper zone on B.Cu, net GND
- added copper zone on F.Cu, net GND
- added copper zone on In1.Cu, net GND
- added copper zone on F.Cu, net V_IN
- removed copper zone on F.Cu, net /SW_BUCK
Other:
- board size 72.2 x 83.5 mm -> 80 x 80 mm

Commit message: ERC errors cleared
Routing:
- net (no net): track 6.69 -> 0.00 mm
- net GND: track 32.3 -> 33.3 mm, vias 171 -> 241

Commit message: added some vias, filled some islands
Routing:
- net GND: track 33.3 -> 34.7 mm, vias 241 -> 286
- net CMD_SD: track 28.8 -> 27.5 mm

Commit message: Readme update
Parts:
- D2: footprint Capacitor_SMD:C_0402_1005Metric_Pad0.74x0.62mm_HandSolder -> telemetry:D20V0L1B2LP-7B
- U3: value LGA14_2P5X3_STM -> ASM330LHHXG1TR
- moved U5 7.19 mm to (85.3, 58.7), turned to 180 degrees
- moved C16 1.67 mm to (87.1, 68.8)
- moved C15 0.90 mm to (83.3, 68.8)
Routing:
- net V_IN: track 59.5 -> 61.2 mm
- net +5V: track 44.1 -> 44.9 mm
- net GND: track 34.7 -> 35.4 mm, vias 286 -> 570
