File: telemetry-kicad/telemetry.kicad_sch (KiCad schematic)
At the start: 118 parts, among them J1 2601-1102, J2 RFPC-SMA27-F, J3 TC2030, J4 2601-1102, J5 2601-1102, J6 USB_C_Receptacle_USB2.0_16P, J7 SD_Card_Receptacle, Q1 DMP3099LQ-7, SW1 SW_NRST, SW2 SW_BOOT0, SW3 CJS-1200TB1, SW4 CJS-1200TB1, U1 LMR33610ADDAR, U10 TLC59108IPWR, U11 MCP1703T-5002E/CB, U13 TXS0108EPW, U2 ASM330LHHXG1TR, U3 LC29HBAMD, U4 TCAN337, U5 STM32H523RCT7, U6 TCAN337, U7 USBLC6-2SC6, U8 TPS2121RUXR, U9 TLC59108IPWR, Y1 ABM8AIG-24.000MHz-8-2Z-T

Commit message: All 3d files added, layout mostly done. some progress routing. schematic is finalised. Switched to microsd card.
Parts:
- removed C37: 10uF, Capacitor_SMD:C_0402_1005Metric_Pad0.74x0.62mm_HandSolder, symbol Device:C
- removed J7: SD_Card_Receptacle, telemetry:SD_Yamaichi_FPS009-4200-0, symbol Connector:SD_Card_Receptacle
- removed R23: 39k, Resistor_SMD:R_0402_1005Metric_Pad0.72x0.64mm_HandSolder, symbol Device:R_US
- removed U11: MCP1703T-5002E/CB, telemetry:MCP1703T-5002E-CB, symbol bspd:MCP1703T-5002E-CB
- added J5: MOLEX_104031-0811, telemetry:MOLEX_104031-0811, symbol telemetry:MOLEX_104031-0811
- added Q2: MMBT3904, Package_TO_SOT_SMD:SOT-23, symbol Transistor_BJT:Q_NPN_BEC
- added R19, R36: 10k, Resistor_SMD:R_0402_1005Metric_Pad0.72x0.64mm_HandSolder, symbol Device:R_US
- added R37: 100k, Resistor_SMD:R_0402_1005Metric_Pad0.72x0.64mm_HandSolder, symbol Device:R_US
- added R38, R39: 39k, Resistor_SMD:R_0402_1005Metric_Pad0.72x0.64mm_HandSolder, symbol Device:R_US
- added U5: LM2940CT-5.0/LF01, telemetry:LM2940CT-5.0-LF01, symbol telemetry:LM2940CT-5.0-LF01
- C16: renamed from C35; value 1uF -> 22uF
- R31: renamed from R28; value 8.66k -> 1.87k
- renumbered C9 to C10, C17 to C11, C10 to C12, C11 to C13, C12 to C14, C32 to C15, C13 to C17, C33 to C18, C34 to C19, C39 to C2, C14 to C20, C15 to C21, C16 to C22, C36 to C23, C28 to C24, C18 to C25, C19 to C26, C20 to C27, C21 to C28, C22 to C29, C2 to C3, C23 to C30, C24 to C31, C25 to C32, C26 to C33, C27 to C34, C29 to C35, C30 to C36, C31 to C37, C3 to C4, C4 to C5, C5 to C6, C6 to C7, C7 to C8, C8 to C9, D6 to D3, D3 to D4, J5 to J6, J6 to J7, LED4 to LED2, LED2 to LED3, LED5 to LED4, LED3 to LED5, R25 to R1, R33 to R10, R35 to R11, R32 to R12, R17 to R13, R16 to R14, R14 to R15, R15 to R16, R19 to R17, R29 to R2, R22 to R20, R4 to R21, R5 to R22, R6 to R23, R13 to R24, R21 to R25, R12 to R26, R7 to R27, R8 to R28, R9 to R29, R31 to R3, R27 to R30, R10 to R32, R11 to R33, R20 to R34, R24 to R35, R1 to R4, R26 to R5, R30 to R6, R2 to R7, R3 to R8, R34 to R9, SW4 to SW1, SW3 to SW2, SW1 to SW3, SW2 to SW4, U3 to U10, U7 to U11, U13 to U12, U8 to U2, U2 to U3, U5 to U6, U6 to U7, U10 to U8
Connections:
- net +12V: now also D1.1 (K), Q1.2 (S); no longer D3.1 (K), J1.1 (1_1), J1.2 (1_2)
- net +3.3V: now also J5.4 (VDD), R19.1
- net +5V: now also U5.3 (OUT)
- net CLK_GNSS: now also U12.14 (B6); no longer U12.17 (B3)
- net CLK_SD: now also J5.5 (CLK)
- net CMD_SD: now also J5.3 (CMD)
- net CS_GNSS: now also U12.13 (B7); no longer U12.16 (B4)
- net D0_SD: now also J5.7 (DAT0)
- net D1_SD: now also J5.8 (DAT1)
- net D2_SD: now also J5.1 (DAT2)
- net D3_SD: now also J5.2 (CD/DAT3)
- net DET_SD: now also J5.9 (DET1), R19.2
- net GND: now also J5.10 (DET2), J5.11 (SH), J5.6 (VSS), Q2.2 (E), R37.2, R38.2, U5.2 (GND)
- net MISO_GNSS: now also U12.15 (B5); no longer U12.18 (B2)
- net MOSI_GNSS: now also U12.16 (B4); no longer U12.20 (B1)
- net TIMERIN_GNSS: now also U12.12 (B8); no longer U12.15 (B5)
- net VDD_EXT: now also R39.1
- net V_IN: now also C15.2, C3.1, C4.1, TP1.1, U1.2 (VIN), U1.3 (EN), U5.1 (IN); no longer F1.1
- net DSEL_1: now reaches U10.5 (D_SEL1)
- net DSEL_1: now also R39.2
- net DSEL_2: now reaches U10.6 (D_SEL2)
- net DSEL_2: now also R38.1
- net CS_GNSS_2V8: now reaches U12.8 (A7)
- net CS_GNSS_2V8: now also U10.18 (I2C_SDA/SPI_CS)
- net TIMERIN_GNSS_2V8: now reaches U12.9 (A8)
- net TIMERIN_GNSS_2V8: now also U10.3 (1PPS)
- net CLK_GNSS_1.8V: no longer names the net of U12.4 (A3)
- net CLK_GNSS_1.8V: no longer U10.19 (I2C_SCL/SPI_CLK)
- net CS_GNSS_1.8V renamed MOSI_GNSS_2V8
- net MOSI_GNSS_2V8: now also U10.21 (RXD1/SPI_MOSI); no longer U10.18 (I2C_SDA/SPI_CS)
- net MISO_GNSS_1.8V: no longer names the net of U12.3 (A2)
- net MISO_GNSS_1.8V: no longer U10.20 (TXD1/SPI_MISO)
- net MOSI_GNSS_1.8V: no longer names the net of U12.1 (A1)
- net MOSI_GNSS_1.8V: no longer U10.21 (RXD1/SPI_MOSI)
- net PG_BUCK: no longer names the net of U6.50 (PA15)
- net RESET_GNSS renamed GNSS_RESET_ASSERT
- net GNSS_RESET_ASSERT: now also R36.1; no longer U12.14 (B6)
- net RESET_GNSS_1.8V renamed CLK_GNSS_2V8
- net CLK_GNSS_2V8: now also U10.19 (I2C_SCL/SPI_CLK); no longer U10.8 (RESET_IN)
- net TIMERIN_GNSS_1.8V renamed MISO_GNSS_2V8
- net MISO_GNSS_2V8: now also U10.20 (TXD1/SPI_MISO); no longer U10.3 (1PPS)
- removed net V_HV: C15.2, C3.1, C4.1, D1.1 (K), Q1.2 (S), TP1.1, U1.2 (VIN), U1.3 (EN)
- new net: Q2.1 (B), R36.2, R37.1
- new net +12V_IN: D3.1 (K), F1.1, J1.1 (1_1), J1.2 (1_2)
- new net GNSS_RESET_N: Q2.3 (C), U10.8 (RESET_N)
- no-connect marks 12 -> 15
Other:
- moved on the sheet: C23, C24, R13, R14, R15, R16, R17, R18, R35, U12

Commit message: Finished all design, no DRC issues. Added BOM, cleaned folder
Parts:
- added H1, H2, H3, H4: MountingHole_Pad, telemetry:MountingHole_3.2mm_M3_Pad, symbol telemetry:MountingHole_Pad
Connections:
- net CAN1+: now also J4.3 (2_1), J4.4 (2_2); no longer J4.1 (1_1), J4.2 (1_2)
- net CAN1-: now also J4.1 (1_1), J4.2 (1_2); no longer J4.3 (2_1), J4.4 (2_2)
- net CAN2+: now also J6.3 (2_1), J6.4 (2_2); no longer J6.1 (1_1), J6.2 (1_2)
- net CAN2-: now also J6.1 (1_1), J6.2 (1_2); no longer J6.3 (2_1), J6.4 (2_2)
- net GND: now also H1.1, H2.1, H3.1, H4.1
Other:
- note added: "Mounting Holes"
