File: hardware/telemetry-kicad/telemetry.kicad_pcb (KiCad board)
At the start: 4 copper layers, 80 x 80 mm, 159 parts, among them J1 2601-1102, J10 RFPC-SMA27-F, J11 MOLEX_104031-0811, J12 Conn_01x04, J2 TC2030, J3 MOLEX_104031-0811, J4 2601-1102, J5 2601-1102, J6 USB_C_Receptacle_USB2.0_16P, J7 RFPC-SMA27-F, J8 RFPC-SMA27-F, J9 RFPC-SMA27-F, Q1 DMP3099LQ-7, Q2 MMBT3904, SW1 CJS-1200TB1, SW2 CJS-1200TB1, SW3 SW_NRST, SW4 SW_BOOT0, U1 LMR33610ADDAR, U10 LC29HEAMD, U11 USBLC6-2SC6, U12 TXS0104EPW, U13 LC29HEAMD, U2 TPS2121RUXR, U3 ASM330LHHXG1TR, U4 TCAN337, U5 LM2940CT-5.0/LF01, U6 STM32H523RCT7, U7 TCAN337, U8 TLC59108IPWR, U9 TLC59108IPWR, Y1 ABM8AIG-24.000MHz-8-2Z-T

Commit message: Update L1 value to 10uH, 16.5m to match the ordered TMPC1265HPV-100MG-D
Parts:
- L1: value 8uH, 14m -> 10uH, 16.5m
Changed lines of the file:
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@@
 			)
 		)
-		(property "Value" "8uH, 14m"
+		(property "Value" "10uH, 16.5m"
 			(at 0 7.4 90)
 			(layer "F.Fab")
